File: MAX31865.kicad_sch (KiCad schematic)
At the start: 16 parts, among them J5 Pt100, U2 MAX31865

Commit message: MAX31865 routed on PCB
Connections:
- net DRDY: no longer names the net of U2.18 (~{DRDY})
- no-connect marks 0 -> 1
Changed lines of the file:
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@@
 		(color 0 0 0 0)
 	)
+	(no_connect
+		(at 121.92 67.31)
+	)
 	(wire
 		(pts
@@
 	(wire
 		(pts
-			(xy 127 138.43) (xy 135.89 138.43)
+			(xy 101.6 100.33) (xy 110.49 100.33)
 		)
 		(stroke
@@
 	(wire
 		(pts
-			(xy 121.92 67.31) (xy 109.22 67.31)
-		)
-		(stroke
-			(width 0.1524)
-			(type solid)
-		)
-	)
-	(wire
-		(pts
 			(xy 153.67 115.57) (xy 153.67 95.25)
 		)
@@
 	(wire
 		(pts
-			(xy 127 133.35) (xy 135.89 133.35)
-		)
-		(stroke
-			(width 0)
-			(type default)
-		)
-	)
-	(wire
-		(pts
-			(xy 127 130.81) (xy 135.89 130.81)
+			(xy 101.6 95.25) (xy 110.49 95.25)
+		)
+		(stroke
+			(width 0)
+			(type default)
+		)
+	)
+	(wire
+		(pts
+			(xy 101.6 92.71) (xy 110.49 92.71)
 		)
 		(stroke
@@
 	(wire
 		(pts
-			(xy 127 135.89) (xy 135.89 135.89)
+			(xy 101.6 97.79) (xy 110.49 97.79)
 		)
 		(stroke
@@
 		)
 	)
-	(label "DRDY"
-		(at 109.22 67.31 0)
-		(fields_autoplaced yes)
-		(effects
-			(font
-				(size 1.2446 1.2446)
-			)
-			(justify left bottom)
-		)
-	)
 	(label "SDO"
 		(at 109.22 77.47 0)
@@
 	)
 	(label "SDO"
-		(at 135.89 133.35 180)
+		(at 110.49 95.25 180)
 		(fields_autoplaced yes)
 		(effects
@@
 	)
 	(label "SDI_5V"
-		(at 135.89 135.89 180)
+		(at 110.49 97.79 180)
 		(fields_autoplaced yes)
 		(effects
@@
 	)
 	(label "CS_5V"
-		(at 135.89 138.43 180)
+		(at 110.49 100.33 180)
 		(fields_autoplaced yes)
 		(effects
@@
 	)
 	(label "SCLK_5V"
-		(at 135.89 130.81 180)
+		(at 110.49 92.71 180)
 		(fields_autoplaced yes)
 		(effects
@@
 	(hierarchical_label "MISO"
 		(shape input)
-		(at 127 133.35 180)
+		(at 101.6 95.25 180)
 		(fields_autoplaced yes)
 		(effects
@@
 	(hierarchical_label "SCK"
 		(shape input)
-		(at 127 130.81 180)
+		(at 101.6 92.71 180)
 		(fields_autoplaced yes)
 		(effects
@@
 	(hierarchical_label "MOSI"
 		(shape input)
-		(at 127 135.89 180)
+		(at 101.6 97.79 180)
 		(fields_autoplaced yes)
 		(effects
@@
 	(hierarchical_label "CS"
 		(shape input)
-		(at 127 138.43 180)
-		(fields_autoplaced yes)
-		(effects
+		(at 101.6 100.33 180)
+		(fields_autoplaced yes)
+		(effects

Commit message: BOM update
Parts:
- D3, D4, D5: Component package type SOD-323 -> (none)
- U2: Component package type 20-TQFN (5x5) -> (none)
Changed lines of the file:
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@@
-			)
-		)
-		(property "Component package type" ""
-			(at 128.27 49.53 0)
-			(effects
-				(font
-					(size 1.27 1.27)
-				)
-				(hide yes)
 			)
 		)
@@
 			)
 		)
-		(property "Component package type" "SOD-323"
-			(at 81.28 76.2 0)
-			(effects
-				(font
-					(size 1.27 1.27)
-				)
-				(hide yes)
-			)
-		)
 		(property "MPN" "1N4148WX-TP"
 			(at 81.28 76.2 0)
@@
 			)
 		)
-		(property "Component package type" ""
-			(at 106.68 62.23 0)
-			(effects
-				(font
-					(size 1.27 1.27)
-				)
-				(hide yes)
-			)
-		)
 		(property "MPN" "/"
 			(at 106.68 62.23 0)
@@
 		)
 		(property "Description" "Solder Jumper, 2-pole, open"
-			(at 182.88 87.63 0)
-			(effects
-				(font
-					(size 1.27 1.27)
-				)
-				(hide yes)
-			)
-		)
-		(property "Component package type" ""
 			(at 182.88 87.63 0)
 			(effects
@@
 			)
 		)
-		(property "Component package type" ""
-			(at 182.88 110.49 0)
-			(effects
-				(font
-					(size 1.27 1.27)
-				)
-				(hide yes)
-			)
-		)
 		(property "MPN" ""
 			(at 182.88 110.49 0)
@@
 			)
 		)
-		(property "Component package type" ""
-			(at 99.06 62.23 0)
-			(effects
-				(font
-					(size 1.27 1.27)
-				)
-				(hide yes)
-			)
-		)
 		(property "MPN" "/"
 			(at 99.06 62.23 0)
@@
 			)
 		)
-		(property "Component package type" ""
-			(at 175.26 71.12 0)
-			(effects
-				(font
-					(size 1.27 1.27)
-				)
-				(hide yes)
-			)
-		)
 		(property "MPN" "/"
 			(at 175.26 71.12 0)
@@
 			)
 		)
-		(property "Component package type" "SOD-323"
-			(at 81.28 72.39 0)
-			(effects
-				(font
-					(size 1.27 1.27)
-				)
-				(hide yes)
-			)
-		)
 		(property "MPN" "1N4148WX-TP"
 			(at 81.28 72.39 0)
@@
 			)
 		)
-		(property "Component package type" ""
-			(at 102.87 55.88 0)
-			(effects
-				(font
-					(size 1.27 1.27)
-				)
-				(hide yes)
-			)
-		)
 		(property "MPN" "/"
 			(at 102.87 55.88 0)
@@
 		)
 		(property "Description" "0.1µF ±10% 50V Ceramic Capacitor X7R 0805 (2012 Metric)"
-			(at 146.05 50.8 0)
-			(effects
-				(font
-					(size 1.27 1.27)
-				)
-				(hide yes)
-			)
-		)
-		(property "Component package type" ""
 			(at 146.05 50.8 0)
 			(effects
@@
 			)
 		)
-		(property "Component package type" ""
-			(at 139.7 41.91 0)
-			(effects
-				(font
-					(size 1.27 1.27)
-				)
-				(hide yes)
-			)
-		)
 		(property "MPN" "LI0805G201R-10"
 			(at 139.7 41.91 0)
@@
 			)
 		)
-		(property "Component package type" ""
-			(at 170.18 100.33 0)
-			(effects
-				(font
-					(size 1.27 1.27)
-				)
-				(hide yes)
-			)
-		)
 		(property "MPN" "/"
 			(at 170.18 100.33 0)
@@
 			)
 		)
-		(property "Component package type" "SOD-323"
-			(at 81.28 68.58 0)
-			(effects
-				(font
-					(size 1.27 1.27)
-				)
-				(hide yes)
-			)
-		)
 		(property "MPN" "1N4148WX-TP"
 			(at 81.28 68.58 0)
@@
 			(at 137.16 82.55 0)
 			(effects
-				(font
-					(size 1.27 1.27)
-				)
-				(hide yes)
-			)
-		)
-		(property "Component package type" "20-TQFN (5x5)"
-			(at 137.16 82.55 0)
-			(effects

Commit message: update README.md
Parts:
- J5: MPN 0393570004 -> 039357-0004
Changed lines of the file:
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@@
 			)
 		)
-		(property "MPN" "0393570004"
+		(property "MPN" "039357-0004"
 			(at 196.85 95.25 0)
 			(effects

Commit message: implemented Eurocircuits design remarks
Parts:
- FB1: footprint Inductor_SMD:L_0805_2012Metric -> external_footprints:LI0805G201R-10
- U2: footprint Package_DFN_QFN:TQFN-20-1EP_5x5mm_P0.65mm_EP3.25x3.25mm -> external_footprints:MAX31865ATP+
Changed lines of the file:
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@@
 			)
 		)
-		(property "Footprint" "Inductor_SMD:L_0805_2012Metric"
+		(property "Footprint" "external_footprints:LI0805G201R-10"
 			(at 141.478 41.91 90)
 			(effects
@@
 			)
 		)
-		(property "Footprint" "Package_DFN_QFN:TQFN-20-1EP_5x5mm_P0.65mm_EP3.25x3.25mm"
+		(property "Footprint" "external_footprints:MAX31865ATP+"
 			(at 140.97 99.06 0)
 			(effects

Commit message: compacter PCB design + debugging improvements pyranometer pin change, AM2315C I2C wiring fix, changed stackup, added ground vias, double sided PCB
Parts:
- renumbered C1 to C11, C2 to C12, C3 to C13, D4 to D10, D5 to D11, D3 to D9, FB1 to FB3, J5 to J9, JP1 to JP7, JP2 to JP8, JP3 to JP9, R4 to R12, R5 to R13, R6 to R14, R7 to R15, U2 to U6
