File: MAX31865.kicad_sch (KiCad schematic)
At the start: 16 parts, among them J9 Pt100, U6 MAX31865

Commit message: build!: upgrade schematic and board to KiCad 10
Parts:
- renumbered C11 to C1, C12 to C2, C13 to C3, D9 to D3, D10 to D4, D11 to D5, FB3 to FB1, J9 to J5, JP7 to JP1, JP8 to JP2, JP9 to JP3, R12 to R4, R13 to R5, R14 to R6, R15 to R7, U6 to U2

Commit message: fix(sch): add PWR_FLAG on +5V, +3.3V, +9V, GND and MAX31865 VDD
Changed lines of the file:
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@@
 	)
 	(junction
+		(at 146.05 45.72)
+		(diameter 0)
+		(color 0 0 0 0)
+	)
+	(junction
 		(at 102.87 74.93)
 		(diameter 0)
@@
 	(wire
 		(pts
+			(xy 153.67 43.18) (xy 153.67 45.72)
+		)
+		(stroke
+			(width 0)
+			(type default)
+		)
+	)
+	(wire
+		(pts
 			(xy 121.92 77.47) (xy 109.22 77.47)
 		)
@@
 	(wire
 		(pts
+			(xy 153.67 45.72) (xy 146.05 45.72)
+		)
+		(stroke
+			(width 0)
+			(type default)
+		)
+	)
+	(wire
+		(pts
 			(xy 139.7 100.33) (xy 139.7 105.41)
 		)
@@
 					(unit 1)
 				)
+			)
+		)
+	)
+	(symbol
+		(lib_id "power:PWR_FLAG")
+		(at 153.67 43.18 0)
+		(unit 1)
+		(body_style 1)
+		(exclude_from_sim no)
+		(in_bom yes)
+		(on_board yes)
+		(in_pos_files yes)
+		(dnp no)
+		(property "Reference" "#FLG04"
+			(at 153.67 41.275 0)
+			(hide yes)
+			(show_name no)
+			(do_not_autoplace no)
+			(effects
+				(font
+					(size 1.27 1.27)
+				)
+			)
+		)
+		(property "Value" "PWR_FLAG"
+			(at 153.67 39.624 0)
+			(show_name no)
+			(do_not_autoplace no)
+			(effects
+				(font
+					(size 1.27 1.27)
+				)
+			)
+		)
+		(property "Footprint" ""
+			(at 153.67 43.18 0)
+			(hide yes)
+			(show_name no)
+			(do_not_autoplace no)
+			(effects
+				(font
+					(size 1.27 1.27)
+				)
+			)
+		)
+		(property "Datasheet" ""
+			(at 153.67 43.18 0)
+			(hide yes)
+			(show_name no)
+			(do_not_autoplace no)
+			(effects
+				(font
+					(size 1.27 1.27)
+				)
+			)
+		)
+		(property "Description" "Special symbol for telling ERC where power comes from"
+			(at 153.67 43.18 0)
+			(hide yes)
+			(show_name no)
+			(do_not_autoplace no)
+			(effects
+				(font
+					(size 1.27 1.27)
+				)
+			)
+		)
+		(pin "1"
+		)
+		(instances
+			(project "testing-station"
+				(path "/ed3950ec-e24f-4dd6-b9cc-eca012f1333b/555649cf-4903-46cd-aa63-9d48293bec40"
+					(reference "#FLG06")
+					(unit 1)
+				)
+				(path "/ed3950ec-e24f-4dd6-b9cc-eca012f1333b/d3c2899f-e06d-436a-b13e-f951511bf9c5"
+					(reference "#FLG04")
+					(unit 1)
+				)
+				(path "/ed3950ec-e24f-4dd6-b9cc-eca012f1333b/e646e214-cec3-4f14-b9f0-d7bac185d28f"
+					(reference "#FLG05")
+					(unit 1)
+				)

Commit message: docs: fill in the title block
Other:
- company: (none) -> UHasselt, Solar Cooker
- title: (none) -> Testing station
Changed lines of the file:
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@@
 	(generator_version "10.0")
 	(paper "A4")
+	(title_block
+		(title "Testing station")
+		(date "2026-10-18")
+		(rev "1.0")
+		(company "UHasselt, Solar Cooker")
+		(comment 1 "Testing station for the solar cooker breakouts")
+		(comment 2 "Design: Lowie Van Vyve")
+		(comment 3 "github.com/solar-cooker-UHasselt/kicad-testing-station")
+	)
 	(text "JP1 to GND for 2/4-wire, to FORCE+ for 3-wire"
 		(exclude_from_sim no)
