File: testing-station.kicad_sch (KiCad schematic)
At the start: 15 parts, among them J1 pyranometer, J10 Conn_01x06_Socket, J11 Conn_01x08_Socket, J2 anemometer, J3 AM2315C, J4 FPC connector, J6 Conn_01x10_Socket, J8 Conn_01x08_Socket, SW1 500SSP1S2M2QEA, U1 TBA_1-0519

Commit message: BOM presets update
Connections:
- net SCA is gone; now on net SDA: J6.2 (Pin_2)
Changed lines of the file:
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@@
 		)
 	)
-	(label "SCA"
+	(label "SDA"
 		(at 228.6 76.2 180)
 		(fields_autoplaced yes)
@@
 		)
 	)
-	(label "SCA"
+	(label "SDA"
 		(at 138.43 62.23 180)
 		(fields_autoplaced yes)

Commit message: compacter PCB design + debugging improvements pyranometer pin change, AM2315C I2C wiring fix, changed stackup, added ground vias, double sided PCB
Parts:
- added TP1: MOSI, TestPoint:TestPoint_Pad_D1.0mm, symbol Connector:TestPoint
- added TP2: MISO, TestPoint:TestPoint_Pad_D1.0mm, symbol Connector:TestPoint
- added TP3: SCK, TestPoint:TestPoint_Pad_D1.0mm, symbol Connector:TestPoint
- added TP4: SDA, TestPoint:TestPoint_Pad_D1.0mm, symbol Connector:TestPoint
- added TP5: SCL, TestPoint:TestPoint_Pad_D1.0mm, symbol Connector:TestPoint
- added TP6: GND, TestPoint:TestPoint_Pad_D1.0mm, symbol Connector:TestPoint
Connections:
- net A5: no longer J1.1 (Pin_1), J10.6 (Pin_6)
- net GND: now also TP6.1
- net MISO: now also TP2.1
- net MOSI: now also TP1.1
- net SCK: now also TP3.1
- net SCL: now also TP5.1
- net SDA: now also TP4.1
- net D10: now reaches J6.8 (Pin_8)
- net D10: now also J1.1 (Pin_1)
