File: testing-station.kicad_sch (KiCad schematic)
At the start: 21 parts, among them J1 pyranometer, J10 Conn_01x06_Socket, J11 Conn_01x08_Socket, J2 anemometer, J3 AM2315C, J4 FPC connector, J6 Conn_01x10_Socket, J8 Conn_01x08_Socket, SW1 500SSP1S2M2QEA, U1 TBA_1-0519

Commit message: fix(sch): turn the unused Arduino pin labels into text
Other:
- note added: "A4"
- note added: "A5"
- note added: "D0"
- note added: "D1"
Changed lines of the file:
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@@
 	(generator_version "10.0")
 	(paper "A4")
+	(text "D0"
+		(exclude_from_sim no)
+		(at 228.6 120.65 0)
+		(effects
+			(font
+				(size 1.27 1.27)
+			)
+			(justify right bottom)
+		)
+	)
+	(text "A5"
+		(exclude_from_sim no)
+		(at 204.47 120.65 0)
+		(effects
+			(font
+				(size 1.27 1.27)
+			)
+			(justify left bottom)
+		)
+	)
+	(text "A4"
+		(exclude_from_sim no)
+		(at 204.47 118.11 0)
+		(effects
+			(font
+				(size 1.27 1.27)
+			)
+			(justify left bottom)
+		)
+	)
+	(text "D1"
+		(exclude_from_sim no)
+		(at 228.6 118.11 0)
+		(effects
+			(font
+				(size 1.27 1.27)
+			)
+			(justify right bottom)
+		)
+	)
 	(junction
 		(at 96.52 100.33)
@@
 		)
 	)
-	(label "D1"
-		(at 228.6 118.11 180)
-		(effects
-			(font
-				(size 1.27 1.27)
-			)
-			(justify right bottom)
-		)
-	)
 	(label "D7"
 		(at 160.02 101.6 0)
@@
 		)
 	)
-	(label "D0"
-		(at 228.6 120.65 180)
-		(effects
-			(font
-				(size 1.27 1.27)
-			)
-			(justify right bottom)
-		)
-	)
 	(label "D2"
 		(at 119.38 115.57 180)
@@
 		)
 	)
-	(label "A4"
-		(at 204.47 118.11 0)
-		(effects
-			(font
-				(size 1.27 1.27)
-			)
-			(justify left bottom)
-		)
-	)
 	(label "SCK"
 		(at 139.7 50.8 180)
@@
 		)
 	)
-	(label "A5"
-		(at 204.47 120.65 0)
-		(effects
-			(font
-				(size 1.27 1.27)
-			)
-			(justify left bottom)
-		)
-	)

Commit message: docs: fill in the title block
Other:
- company: (none) -> UHasselt, Solar Cooker
- title: (none) -> Testing station
Changed lines of the file:
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@@
 	(generator_version "10.0")
 	(paper "A4")
+	(title_block
+		(title "Testing station")
+		(date "2026-10-18")
+		(rev "1.0")
+		(company "UHasselt, Solar Cooker")
+		(comment 1 "Testing station for the solar cooker breakouts")
+		(comment 2 "Design: Lowie Van Vyve")
+		(comment 3 "github.com/solar-cooker-UHasselt/kicad-testing-station")
+	)
 	(text "D0"
 		(exclude_from_sim no)
