File: BME680.kicad_sch (KiCad schematic)
At the start: 12 parts, among them IC1 BME680, Q1 BSS138

Commit message: docs: fill in the title block
Other:
- company: (none) -> UHasselt, Solar Cooker
- title: (none) -> Testing station
Changed lines of the file:
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@@
 	(generator_version "10.0")
 	(paper "A4")
+	(title_block
+		(title "Testing station")
+		(date "2026-10-18")
+		(rev "1.0")
+		(company "UHasselt, Solar Cooker")
+		(comment 1 "Testing station for the solar cooker breakouts")
+		(comment 2 "Design: Lowie Van Vyve")
+		(comment 3 "github.com/solar-cooker-UHasselt/kicad-testing-station")
+	)
 	(text "I2C Pullups"
 		(exclude_from_sim no)
